File: 4. Ročník/ELEKTRO/PCB/PCB.kicad_sch (KiCad schematic)
At the start: 19 parts, among them J1 Conn_01x04, J10 Motor_Right, J11 Jetson Pinout, J12 Screw_Terminal_01x02, J13 Screw_Terminal_01x02, J14 Screw_Terminal_01x02, J15 Napajeni BTS_R, J16 Napajeni BTS_L, J2 BX100 Alarm, J3 Conn_01x08, J4 BTS_Napajeni, J5 BTS_K_Motoru, J6 BTS_Napajeni, J7 BTS_K_Motoru, J8 Conn_01x08, J9 Motor_Left, SW1 SW_SPST

Commit message: PCB v1.0 fixes: 0.4/0.8mm routing, GND plane pour, silkscreen updates
Parts:
- added C1: 1000uF / 35V, Capacitor_THT:CP_Radial_D10.0mm_P5.00mm, symbol Device:C_Polarized
- added D1: LED, LED_THT:LED_D3.0mm, symbol Device:LED
- added H1, H2, H3, H4: MountingHole, MountingHole:MountingHole_3.2mm_M3, symbol Mechanical:MountingHole
- added J17, J18: Conn_01x04, Connector_PinHeader_2.54mm:PinHeader_1x04_P2.54mm_Vertical, symbol Connector_Generic:Conn_01x04
- added R1: 1k, Resistor_THT:R_Axial_DIN0207_L6.3mm_D2.5mm_P10.16mm_Horizontal, symbol Device:R
Connections:
- net +12V: now also SW1.1 (A), C1.1, R1.2
- net +3V3: now also J17.3 (Pin_3), J18.3 (Pin_3)
- net GND: now also C1.2, D1.1 (K), J17.4 (Pin_4), J18.4 (Pin_4)
- net MOTOR_L_ENK_A: now also J18.1 (Pin_1)
- net MOTOR_L_ENK_B: now also J18.2 (Pin_2)
- net MOTOR_R_ENK_A: now also J17.1 (Pin_1)
- net MOTOR_R_ENK_B: now also J17.2 (Pin_2)
- new net: D1.2 (A), R1.1
Other:
- moved on the sheet: BT1, F1, J1, J2, SW1
